File: Mikrobus-Proto-18.sch (EAGLE design)
At the start: 38 parts

Commit message: Add Ground Plane
Connections:
- removed net N$21: JP8.1, JP8.2, JP8.3, JP9.1, JP9.2, JP9.3, MB1.GND@1, MB1.GND@2, U$3.P$1, U$3.P$2, U$3.P$3, U$3.P$4, U$3.P$5, U$3.P$6, U$3.P$7, U$3.P$8, U$3.P$9
- removed net N$46: U$18.P$1, U$18.P$2, U$18.P$3, U$18.P$4
- new net GND: JP8.1, JP8.2, JP8.3, JP9.1, JP9.2, JP9.3, MB1.GND@1, MB1.GND@2, U$18.P$1, U$18.P$2, U$18.P$3, U$18.P$4, U$3.P$1, U$3.P$2, U$3.P$3, U$3.P$4, U$3.P$5, U$3.P$6, U$3.P$7, U$3.P$8, U$3.P$9

Commit message: Signal names changed for preperation of Fritzing parts
Connections:
- net N$1 renamed INT
- net N$11 renamed MISO
- net N$13 renamed AN
- net N$15 renamed MOSI
- net N$2 renamed +5V
- net N$24 renamed PWM
- net N$26 renamed TX
- net N$29 renamed RX
- net N$32 renamed SDA
- net N$35 renamed SCL
- net N$4 renamed +3.3V
- net N$43 renamed RST
- net N$48 renamed SCK
- net N$5 renamed CS
Changed lines of the file:
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@@
 </busses>
 <nets>
-<net name="N$13" class="0">
+<net name="AN" class="0">
 <segment>
 <pinref part="JP1" gate="G$1" pin="3"/>
@@
 </segment>
 </net>
-<net name="N$1" class="0">
+<net name="INT" class="0">
 <segment>
 <pinref part="JP16" gate="G$1" pin="1"/>
@@
 </segment>
 </net>
-<net name="N$5" class="0">
+<net name="CS" class="0">
 <segment>
 <pinref part="JP3" gate="G$1" pin="2"/>
@@
 </segment>
 </net>
-<net name="N$11" class="0">
+<net name="MISO" class="0">
 <segment>
 <pinref part="JP5" gate="G$1" pin="2"/>
@@
 </segment>
 </net>
-<net name="N$15" class="0">
+<net name="MOSI" class="0">
 <segment>
 <pinref part="JP6" gate="G$1" pin="2"/>
@@
 </segment>
 </net>
-<net name="N$24" class="0">
+<net name="PWM" class="0">
 <segment>
 <pinref part="JP15" gate="G$1" pin="2"/>
@@
 </segment>
 </net>
-<net name="N$26" class="0">
+<net name="TX" class="0">
 <segment>
 <pinref part="JP13" gate="G$1" pin="1"/>
@@
 </segment>
 </net>
-<net name="N$29" class="0">
+<net name="RX" class="0">
 <segment>
 <pinref part="JP14" gate="G$1" pin="1"/>
@@
 </segment>
 </net>
-<net name="N$32" class="0">
+<net name="SDA" class="0">
 <segment>
 <pinref part="JP11" gate="G$1" pin="1"/>
@@
 </segment>
 </net>
-<net name="N$35" class="0">
+<net name="SCL" class="0">
 <segment>
 <pinref part="JP12" gate="G$1" pin="1"/>
@@
 </segment>
 </net>
-<net name="N$4" class="0">
+<net name="+3.3V" class="0">
 <segment>
 <pinref part="JP7" gate="G$1" pin="1"/>
@@
 </segment>
 </net>
-<net name="N$43" class="0">
+<net name="RST" class="0">
 <segment>
 <pinref part="JP2" gate="G$1" pin="1"/>
@@
 </segment>
 </net>
-<net name="N$48" class="0">
+<net name="SCK" class="0">
 <segment>
 <pinref part="JP4" gate="G$1" pin="1"/>
@@
 </segment>
 </net>
-<net name="N$2" class="0">
+<net name="+5V" class="0">
 <segment>
 <pinref part="MB1" gate="G$1" pin="+5V"/>

Commit message: Better Fritzing part thanks to Steve Lilley
Connections:
- net N$12 renamed R8
- net N$16 renamed L7
- net N$17 renamed R7
- net N$19 renamed L6
- net N$20 renamed R6
- net N$22 renamed R9
- net N$25 renamed L8
- net N$28 renamed L5
- net N$31 renamed R5
- net N$34 renamed L4
- net N$37 renamed R4
- net N$38 renamed L3
- net N$40 renamed R3
- net N$44 renamed L2
- net N$45 renamed R2
- net N$47 renamed R1
- net N$9 renamed L9
- new net L1: U$18.P$1, U$18.P$2, U$18.P$3, U$18.P$4
- net GND: no longer U$18.P$1, U$18.P$2, U$18.P$3, U$18.P$4
Changed lines of the file:
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@@
 </segment>
 </net>
-<net name="N$9" class="0">
+<net name="L9" class="0">
 <segment>
 <pinref part="U$4" gate="G$1" pin="P$1"/>
@@
 </segment>
 </net>
-<net name="N$12" class="0">
+<net name="R8" class="0">
 <segment>
 <pinref part="U$7" gate="G$1" pin="P$1"/>
@@
 </segment>
 </net>
-<net name="N$16" class="0">
+<net name="L7" class="0">
 <segment>
 <pinref part="U$8" gate="G$1" pin="P$1"/>
@@
 </segment>
 </net>
-<net name="N$17" class="0">
+<net name="R7" class="0">
 <segment>
 <pinref part="U$9" gate="G$1" pin="P$1"/>
@@
 </segment>
 </net>
-<net name="N$19" class="0">
+<net name="L6" class="0">
 <segment>
 <pinref part="U$10" gate="G$1" pin="P$1"/>
@@
 </segment>
 </net>
-<net name="N$20" class="0">
+<net name="R6" class="0">
 <segment>
 <pinref part="U$11" gate="G$1" pin="P$1"/>
@@
 </segment>
 </net>
-<net name="N$22" class="0">
+<net name="R9" class="0">
 <segment>
 <pinref part="U$5" gate="G$1" pin="P$1"/>
@@
 </segment>
 </net>
-<net name="N$25" class="0">
+<net name="L8" class="0">
 <segment>
 <pinref part="U$6" gate="G$1" pin="P$1"/>
@@
 </segment>
 </net>
-<net name="N$28" class="0">
+<net name="L5" class="0">
 <segment>
 <pinref part="U$12" gate="G$1" pin="P$1"/>
@@
 </segment>
 </net>
-<net name="N$31" class="0">
+<net name="R5" class="0">
 <segment>
 <pinref part="U$13" gate="G$1" pin="P$1"/>
@@
 </segment>
 </net>
-<net name="N$34" class="0">
+<net name="L4" class="0">
 <segment>
 <pinref part="U$14" gate="G$1" pin="P$1"/>
@@
 </segment>
 </net>
-<net name="N$37" class="0">
+<net name="R4" class="0">
 <segment>
 <pinref part="U$15" gate="G$1" pin="P$1"/>
@@
 </segment>
 </net>
-<net name="N$38" class="0">
+<net name="L3" class="0">
 <segment>
 <pinref part="U$16" gate="G$1" pin="P$1"/>
@@
 </segment>
 </net>
-<net name="N$40" class="0">
+<net name="R3" class="0">
 <segment>
 <pinref part="U$17" gate="G$1" pin="P$1"/>
@@
 </segment>
 </net>
-<net name="N$44" class="0">
+<net name="L2" class="0">
 <segment>
 <pinref part="U$1" gate="G$1" pin="P$1"/>
@@
 </segment>
 </net>
-<net name="N$45" class="0">
+<net name="R2" class="0">
 <segment>
 <pinref part="U$2" gate="G$1" pin="P$1"/>
@@
 </segment>
 </net>
-<net name="GND" class="0">
+<net name="L1" class="0">
 <segment>
 <pinref part="U$18" gate="G$1" pin="P$1"/>
@@
 <junction x="5.08" y="116.84"/>
 </segment>
+</net>
+<net name="R1" class="0">
+<segment>
+<pinref part="U$19" gate="G$1" pin="P$1"/>
+<pinref part="U$19" gate="G$1" pin="P$4"/>
+<wire x1="17.78" y1="124.46" x2="17.78" y2="121.92" width="0.1524" layer="91"/>
+<junction x="17.78" y="124.46"/>
+<pinref part="U$19" gate="G$1" pin="P$2"/>
+<junction x="17.78" y="121.92"/>
+<wire x1="17.78" y1="121.92" x2="17.78" y2="119.38" width="0.1524" layer="91"/>
+<pinref part="U$19" gate="G$1" pin="P$3"/>
+<junction x="17.78" y="119.38"/>
+<wire x1="17.78" y1="119.38" x2="17.78" y2="116.84" width="0.1524" layer="91"/>
+<junction x="17.78" y="116.84"/>
+</segment>
+</net>
+<net name="RST" class="0">
+<segment>
+<pinref part="JP2" gate="G$1" pin="1"/>
+<pinref part="JP2" gate="G$1" pin="2"/>
+<wire x1="35.56" y1="33.02" x2="38.1" y2="33.02" width="0.1524" layer="91"/>
+<pinref part="JP2" gate="G$1" pin="3"/>
+<wire x1="40.64" y1="33.02" x2="50.8" y2="33.02" width="0.1524" layer="91"/>
+<wire x1="50.8" y1="33.02" x2="50.8" y2="22.86" width="0.1524" layer="91"/>
+<wire x1="50.8" y1="22.86" x2="53.34" y2="22.86" width="0.1524" layer="91"/>
+<pinref part="MB1" gate="G$1" pin="RST"/>
+<junction x="53.34" y="22.86"/>
+<wire x1="38.1" y1="33.02" x2="40.64" y2="33.02" width="0.1524" layer="91"/>
+<junction x="35.56" y="33.02"/>
+<junction x="38.1" y="33.02"/>
+<junction x="40.64" y="33.02"/>
+</segment>
+</net>
+<net name="SCK" class="0">
+<segment>
+<pinref part="JP4" gate="G$1" pin="1"/>
+<pinref part="JP4" gate="G$1" pin="2"/>
+<wire x1="35.56" y1="17.78" x2="38.1" y2="17.78" width="0.1524" layer="91"/>
+<pinref part="JP4" gate="G$1" pin="3"/>
+<wire x1="40.64" y1="17.78" x2="53.34" y2="17.78" width="0.1524" layer="91"/>
+<pinref part="MB1" gate="G$1" pin="SCK"/>
+<junction x="53.34" y="17.78"/>
+<wire x1="38.1" y1="17.78" x2="40.64" y2="17.78" width="0.1524" layer="91"/>
+<junction x="35.56" y="17.78"/>
+<junction x="38.1" y="17.78"/>
+<junction x="40.64" y="17.78"/>
+</segment>
+</net>
+<net name="+5V" class="0">
+<segment>
+<pinref part="MB1" gate="G$1" pin="+5V"/>
+<junction x="83.82" y="10.16"/>
+<wire x1="86.36" y1="10.16" x2="83.82" y2="10.16" width="0.1524" layer="91"/>
+<pinref part="JP10" gate="G$1" pin="1"/>
+<wire x1="116.84" y1="-12.7" x2="111.76" y2="-12.7" width="0.1524" layer="91"/>
+<wire x1="111.76" y1="-12.7" x2="111.76" y2="-15.24" width="0.1524" layer="91"/>
+<wire x1="111.76" y1="-15.24" x2="86.36" y2="-15.24" width="0.1524" layer="91"/>
+<wire x1="86.36" y1="-15.24" x2="86.36" y2="10.16" width="0.1524" layer="91"/>
+<pinref part="JP10" gate="G$1" pin="2"/>
+<junction x="119.38" y="-12.7"/>
+<wire x1="116.84" y1="-12.7" x2="119.38" y2="-12.7" width="0.1524" layer="91"/>
+<pinref part="JP10" gate="G$1" pin="3"/>
+<wire x1="121.92" y1="-12.7" x2="134.62" y2="-12.7" width="0.1524" layer="91"/>
+<wire x1="134.62" y1="-12.7" x2="134.62" y2="66.04" width="0.1524" layer="91"/>
+<pinref part="JP18" gate="G$1" pin="1"/>
+<wire x1="73.66" y1="66.04" x2="76.2" y2="66.04" width="0.1524" layer="91"/>
+<wire x1="76.2" y1="66.04" x2="78.74" y2="66.04" width="0.1524" layer="91"/>
+<wire x1="78.74" y1="66.04" x2="134.62" y2="66.04" width="0.1524" layer="91"/>
+<junction x="73.66" y="66.04"/>
+<pinref part="JP18" gate="G$1" pin="2"/>
+<junction x="76.2" y="66.04"/>
+<pinref part="JP18" gate="G$1" pin="3"/>
+<junction x="78.74" y="66.04"/>
+<wire x1="119.38" y1="-12.7" x2="121.92" y2="-12.7" width="0.1524" layer="91"/>
+<junction x="116.84" y="-12.7"/>
+<junction x="121.92" y="-12.7"/>
+</segment>
+</net>
+<net name="GND" class="0">
 <segment>
 <pinref part="JP8" gate="G$1" pin="2"/>
@@
 </segment>
 </net>
-<net name="N$47" class="0">
-<segment>
-<pinref part="U$19" gate="G$1" pin="P$1"/>
-<pinref part="U$19" gate="G$1" pin="P$4"/>
-<wire x1="17.78" y1="124.46" x2="17.78" y2="121.92" width="0.1524" layer="91"/>
-<junction x="17.78" y="124.46"/>
-<pinref part="U$19" gate="G$1" pin="P$2"/>
-<junction x="17.78" y="121.92"/>
-<wire x1="17.78" y1="121.92" x2="17.78" y2="119.38" width="0.1524" layer="91"/>
-<pinref part="U$19" gate="G$1" pin="P$3"/>
-<junction x="17.78" y="119.38"/>
-<wire x1="17.78" y1="119.38" x2="17.78" y2="116.84" width="0.1524" layer="91"/>
-<junction x="17.78" y="116.84"/>
-</segment>
-</net>
-<net name="RST" class="0">
-<segment>
-<pinref part="JP2" gate="G$1" pin="1"/>
-<pinref part="JP2" gate="G$1" pin="2"/>
-<wire x1="35.56" y1="33.02" x2="38.1" y2="33.02" width="0.1524" layer="91"/>
-<pinref part="JP2" gate="G$1" pin="3"/>
-<wire x1="40.64" y1="33.02" x2="50.8" y2="33.02" width="0.1524" layer="91"/>
-<wire x1="50.8" y1="33.02" x2="50.8" y2="22.86" width="0.1524" layer="91"/>
-<wire x1="50.8" y1="22.86" x2="53.34" y2="22.86" width="0.1524" layer="91"/>
-<pinref part="MB1" gate="G$1" pin="RST"/>
-<junction x="53.34" y="22.86"/>
-<wire x1="38.1" y1="33.02" x2="40.64" y2="33.02" width="0.1524" layer="91"/>
-<junction x="35.56" y="33.02"/>
-<junction x="38.1" y="33.02"/>
-<junction x="40.64" y="33.02"/>
-</segment>
-</net>
-<net name="SCK" class="0">
-<segment>
-<pinref part="JP4" gate="G$1" pin="1"/>
-<pinref part="JP4" gate="G$1" pin="2"/>
-<wire x1="35.56" y1="17.78" x2="38.1" y2="17.78" width="0.1524" layer="91"/>
-<pinref part="JP4" gate="G$1" pin="3"/>
-<wire x1="40.64" y1="17.78" x2="53.34" y2="17.78" width="0.1524" layer="91"/>
-<pinref part="MB1" gate="G$1" pin="SCK"/>
-<junction x="53.34" y="17.78"/>
-<wire x1="38.1" y1="17.78" x2="40.64" y2="17.78" width="0.1524" layer="91"/>
-<junction x="35.56" y="17.78"/>
-<junction x="38.1" y="17.78"/>
-<junction x="40.64" y="17.78"/>
-</segment>
-</net>
-<net name="+5V" class="0">
-<segment>
-<pinref part="MB1" gate="G$1" pin="+5V"/>
-<junction x="83.82" y="10.16"/>
-<wire x1="86.36" y1="10.16" x2="83.82" y2="10.16" width="0.1524" layer="91"/>
-<pinref part="JP10" gate="G$1" pin="1"/>
-<wire x1="116.84" y1="-12.7" x2="111.76" y2="-12.7" width="0.1524" layer="91"/>
-<wire x1="111.76" y1="-12.7" x2="111.76" y2="-15.24" width="0.1524" layer="91"/>
-<wire x1="111.76" y1="-15.24" x2="86.36" y2="-15.24" width="0.1524" layer="91"/>
-<wire x1="86.36" y1="-15.24" x2="86.36" y2="10.16" width="0.1524" layer="91"/>
-<pinref part="JP10" gate="G$1" pin="2"/>
-<junction x="119.38" y="-12.7"/>
-<wire x1="116.84" y1="-12.7" x2="119.38" y2="-12.7" width="0.1524" layer="91"/>
-<pinref part="JP10" gate="G$1" pin="3"/>
-<wire x1="121.92" y1="-12.7" x2="134.62" y2="-12.7" width="0.1524" layer="91"/>
-<wire x1="134.62" y1="-12.7" x2="134.62" y2="66.04" width="0.1524" layer="91"/>
-<pinref part="JP18" gate="G$1" pin="1"/>
-<wire x1="73.66" y1="66.04" x2="76.2" y2="66.04" width="0.1524" layer="91"/>
-<wire x1="76.2" y1="66.04" x2="78.74" y2="66.04" width="0.1524" layer="91"/>
-<wire x1="78.74" y1="66.04" x2="134.62" y2="66.04" width="0.1524" layer="91"/>
-<junction x="73.66" y="66.04"/>
-<pinref part="JP18" gate="G$1" pin="2"/>
-<junction x="76.2" y="66.04"/>
-<pinref part="JP18" gate="G$1" pin="3"/>
-<junction x="78.74" y="66.04"/>
-<wire x1="119.38" y1="-12.7" x2="121.92" y2="-12.7" width="0.1524" layer="91"/>
-<junction x="116.84" y="-12.7"/>
-<junction x="121.92" y="-12.7"/>
-</segment>
-</net>
