File: Mikrobus-Proto-22.brd (EAGLE design)
At the start: 27.9 x 57.1 mm, 39 parts

Commit message: Signal names changed for preperation of Fritzing parts
Connections:
- net N$1 renamed INT
- net N$11 renamed MISO
- net N$13 renamed AN
- net N$15 renamed MOSI
- net N$2 renamed +5V
- net N$24 renamed PWM
- net N$26 renamed TX
- net N$29 renamed RX
- net N$32 renamed SDA
- net N$35 renamed SCL
- net N$4 renamed +3.3V
- net N$43 renamed RST
- net N$48 renamed SCK
- net N$5 renamed CS
Changed lines of the file:
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@@
 </elements>
 <signals>
-<signal name="N$13">
+<signal name="AN">
 <contactref element="JP1" pad="3"/>
 <contactref element="MB1" pad="1"/>
@@
 <wire x1="7.62" y1="22.86" x2="5.08" y2="22.86" width="0.1524" layer="1"/>
 </signal>
-<signal name="N$1">
+<signal name="INT">
 <contactref element="JP16" pad="1"/>
 <contactref element="MB1" pad="15"/>
@@
 <wire x1="20.32" y1="20.32" x2="22.86" y2="20.32" width="0.1524" layer="1"/>
 </signal>
-<signal name="N$5">
+<signal name="CS">
 <contactref element="JP3" pad="2"/>
 <contactref element="JP3" pad="1"/>
@@
 <wire x1="7.62" y1="17.78" x2="10.16" y2="17.78" width="0.1524" layer="1"/>
 </signal>
-<signal name="N$11">
+<signal name="MISO">
 <contactref element="JP5" pad="2"/>
 <contactref element="JP5" pad="1"/>
@@
 <wire x1="7.62" y1="12.7" x2="10.16" y2="12.7" width="0.1524" layer="1"/>
 </signal>
-<signal name="N$15">
+<signal name="MOSI">
 <contactref element="JP6" pad="2"/>
 <contactref element="JP6" pad="1"/>
@@
 <wire x1="7.62" y1="10.16" x2="10.16" y2="10.16" width="0.1524" layer="1"/>
 </signal>
-<signal name="N$24">
+<signal name="PWM">
 <contactref element="JP15" pad="2"/>
 <contactref element="MB1" pad="16"/>
@@
 <wire x1="20.32" y1="22.86" x2="22.86" y2="22.86" width="0.1524" layer="1"/>
 </signal>
-<signal name="N$26">
+<signal name="TX">
 <contactref element="JP13" pad="1"/>
 <contactref element="MB1" pad="13"/>
@@
 <wire x1="20.32" y1="15.24" x2="22.86" y2="15.24" width="0.1524" layer="1"/>
 </signal>
-<signal name="N$29">
+<signal name="RX">
 <contactref element="JP14" pad="1"/>
 <contactref element="MB1" pad="14"/>
@@
 <wire x1="20.32" y1="17.78" x2="22.86" y2="17.78" width="0.1524" layer="1"/>
 </signal>
-<signal name="N$32">
+<signal name="SDA">
 <contactref element="JP11" pad="1"/>
 <contactref element="MB1" pad="11"/>
@@
 <wire x1="20.32" y1="10.16" x2="22.86" y2="10.16" width="0.1524" layer="1"/>
 </signal>
-<signal name="N$35">
+<signal name="SCL">
 <contactref element="JP12" pad="1"/>
 <contactref element="MB1" pad="12"/>
@@
 <wire x1="20.32" y1="12.7" x2="22.86" y2="12.7" width="0.1524" layer="1"/>
 </signal>
-<signal name="N$4">
+<signal name="+3.3V">
 <contactref element="JP7" pad="1"/>
 <contactref element="JP7" pad="2"/>
@@
 </polygon>
 </signal>
-<signal name="N$43">
+<signal name="RST">
 <contactref element="JP2" pad="1"/>
 <contactref element="JP2" pad="2"/>
@@
 <wire x1="7.62" y1="20.32" x2="10.16" y2="20.32" width="0.1524" layer="1"/>
 </signal>
-<signal name="N$48">
+<signal name="SCK">
 <contactref element="JP4" pad="1"/>
 <contactref element="JP4" pad="2"/>
@@
 <wire x1="7.62" y1="15.24" x2="10.16" y2="15.24" width="0.1524" layer="1"/>
 </signal>
-<signal name="N$2">
+<signal name="+5V">
 <contactref element="JP10" pad="1"/>
 <contactref element="MB1" pad="10"/>

Commit message: Better Fritzing part thanks to Steve Lilley
Connections:
- net N$10 renamed R5
- net N$12 renamed L7
- net N$14 renamed R4
- net N$16 renamed L8
- net N$17 renamed L6
- net N$18 renamed R1
- net N$19 renamed R3
- net N$20 renamed R2
- net N$21 renamed R7
- net N$22 renamed L11
- net N$23 renamed R8
- net N$25 renamed L9
- net N$27 renamed R9
- net N$28 renamed R10
- net N$3 renamed L3
- net N$30 renamed R11
- net N$44 renamed L4
- net N$45 renamed L5
- net N$6 renamed L2
- net N$7 renamed L1
- net N$8 renamed R6
- net N$9 renamed L10
Changed lines of the file:
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@@
 <wire x1="7.62" y1="7.62" x2="10.16" y2="7.62" width="0.1524" layer="1"/>
 </signal>
-<signal name="N$9">
+<signal name="L10">
 <contactref element="U$4" pad="1"/>
 <contactref element="U$4" pad="4"/>
@@
 <wire x1="7.62" y1="33.02" x2="10.16" y2="33.02" width="0.1524" layer="1"/>
 </signal>
-<signal name="N$12">
+<signal name="L7">
 <contactref element="U$7" pad="1"/>
 <contactref element="U$7" pad="4"/>
@@
 <wire x1="7.62" y1="40.64" x2="10.16" y2="40.64" width="0.1524" layer="1"/>
 </signal>
-<signal name="N$16">
+<signal name="L8">
 <contactref element="U$8" pad="1"/>
 <contactref element="U$8" pad="4"/>
@@
 <wire x1="7.62" y1="38.1" x2="10.16" y2="38.1" width="0.1524" layer="1"/>
 </signal>
-<signal name="N$17">
+<signal name="L6">
 <contactref element="U$9" pad="1"/>
 <contactref element="U$9" pad="4"/>
@@
 <wire x1="7.62" y1="43.18" x2="10.16" y2="43.18" width="0.1524" layer="1"/>
 </signal>
-<signal name="N$22">
+<signal name="L11">
 <contactref element="U$5" pad="1"/>
 <contactref element="U$5" pad="4"/>
@@
 <wire x1="7.62" y1="30.48" x2="10.16" y2="30.48" width="0.1524" layer="1"/>
 </signal>
-<signal name="N$25">
+<signal name="L9">
 <contactref element="U$6" pad="1"/>
 <contactref element="U$6" pad="4"/>
@@
 <wire x1="7.62" y1="35.56" x2="10.16" y2="35.56" width="0.1524" layer="1"/>
 </signal>
-<signal name="N$44">
+<signal name="L4">
 <contactref element="U$1" pad="1"/>
 <contactref element="U$1" pad="4"/>
@@
 <wire x1="7.62" y1="48.26" x2="10.16" y2="48.26" width="0.1524" layer="1"/>
 </signal>
-<signal name="N$45">
+<signal name="L5">
 <contactref element="U$2" pad="1"/>
 <contactref element="U$2" pad="4"/>
@@
 <wire x1="20.32" y1="7.62" x2="22.86" y2="7.62" width="0.1524" layer="1"/>
 </signal>
-<signal name="N$3">
+<signal name="L3">
 <contactref element="U$3" pad="1"/>
 <contactref element="U$3" pad="2"/>
@@
 <wire x1="7.62" y1="50.8" x2="10.16" y2="50.8" width="0.1524" layer="1"/>
 </signal>
-<signal name="N$6">
+<signal name="L2">
 <contactref element="U$10" pad="1"/>
 <contactref element="U$10" pad="2"/>
@@
 <wire x1="7.62" y1="53.34" x2="10.16" y2="53.34" width="0.1524" layer="1"/>
 </signal>
-<signal name="N$7">
+<signal name="L1">
 <contactref element="U$11" pad="1"/>
 <contactref element="U$11" pad="2"/>
@@
 <wire x1="7.62" y1="55.88" x2="10.16" y2="55.88" width="0.1524" layer="1"/>
 </signal>
-<signal name="N$8">
+<signal name="R6">
 <contactref element="JP22" pad="5"/>
 <contactref element="JP22" pad="4"/>
@@
 <wire x1="22.86" y1="43.18" x2="25.4" y2="43.18" width="0.1524" layer="1"/>
 </signal>
-<signal name="N$10">
+<signal name="R5">
 <contactref element="JP23" pad="5"/>
 <contactref element="JP23" pad="4"/>
@@
 <wire x1="22.86" y1="45.72" x2="25.4" y2="45.72" width="0.1524" layer="1"/>
 </signal>
-<signal name="N$14">
+<signal name="R4">
 <contactref element="JP24" pad="5"/>
 <contactref element="JP24" pad="4"/>
@@
 <wire x1="22.86" y1="48.26" x2="25.4" y2="48.26" width="0.1524" layer="1"/>
 </signal>
-<signal name="N$18">
+<signal name="R1">
 <contactref element="JP27" pad="5"/>
 <contactref element="JP27" pad="4"/>
@@
 <wire x1="22.86" y1="55.88" x2="25.4" y2="55.88" width="0.1524" layer="1"/>
 </signal>
-<signal name="N$19">
+<signal name="R3">
 <contactref element="JP25" pad="5"/>
 <contactref element="JP25" pad="4"/>
@@
 <wire x1="22.86" y1="50.8" x2="25.4" y2="50.8" width="0.1524" layer="1"/>
 </signal>
-<signal name="N$20">
+<signal name="R2">
 <contactref element="JP26" pad="5"/>
 <contactref element="JP26" pad="4"/>
@@
 <wire x1="22.86" y1="53.34" x2="25.4" y2="53.34" width="0.1524" layer="1"/>
 </signal>
-<signal name="N$21">
+<signal name="R7">
 <contactref element="JP21" pad="5"/>
 <contactref element="JP21" pad="4"/>
@@
 <wire x1="22.86" y1="40.64" x2="25.4" y2="40.64" width="0.1524" layer="1"/>
 </signal>
-<signal name="N$23">
+<signal name="R8">
 <contactref element="JP20" pad="5"/>
 <contactref element="JP20" pad="4"/>
@@
 <wire x1="22.86" y1="38.1" x2="25.4" y2="38.1" width="0.1524" layer="1"/>
 </signal>
-<signal name="N$27">
+<signal name="R9">
 <contactref element="JP19" pad="5"/>
 <contactref element="JP19" pad="4"/>
@@
 <wire x1="22.86" y1="35.56" x2="25.4" y2="35.56" width="0.1524" layer="1"/>
 </signal>
-<signal name="N$28">
+<signal name="R10">
 <contactref element="JP18" pad="5"/>
 <contactref element="JP18" pad="4"/>
@@
 <wire x1="22.86" y1="33.02" x2="25.4" y2="33.02" width="0.1524" layer="1"/>
 </signal>
-<signal name="N$30">
+<signal name="R11">
 <contactref element="JP17" pad="5"/>
 <contactref element="JP17" pad="4"/>
