File: Mikrobus-Proto-22.sch (EAGLE design)
At the start: 39 parts

Commit message: Signal names changed for preperation of Fritzing parts
Connections:
- net N$1 renamed INT
- net N$11 renamed MISO
- net N$13 renamed AN
- net N$15 renamed MOSI
- net N$2 renamed +5V
- net N$24 renamed PWM
- net N$26 renamed TX
- net N$29 renamed RX
- net N$32 renamed SDA
- net N$35 renamed SCL
- net N$4 renamed +3.3V
- net N$43 renamed RST
- net N$48 renamed SCK
- net N$5 renamed CS
Changed lines of the file:
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@@
 </busses>
 <nets>
-<net name="N$13" class="0">
+<net name="AN" class="0">
 <segment>
 <pinref part="JP1" gate="G$1" pin="3"/>
@@
 </segment>
 </net>
-<net name="N$1" class="0">
+<net name="INT" class="0">
 <segment>
 <pinref part="JP16" gate="G$1" pin="1"/>
@@
 </segment>
 </net>
-<net name="N$5" class="0">
+<net name="CS" class="0">
 <segment>
 <pinref part="JP3" gate="G$1" pin="2"/>
@@
 </segment>
 </net>
-<net name="N$11" class="0">
+<net name="MISO" class="0">
 <segment>
 <pinref part="JP5" gate="G$1" pin="2"/>
@@
 </segment>
 </net>
-<net name="N$15" class="0">
+<net name="MOSI" class="0">
 <segment>
 <pinref part="JP6" gate="G$1" pin="2"/>
@@
 </segment>
 </net>
-<net name="N$24" class="0">
+<net name="PWM" class="0">
 <segment>
 <pinref part="JP15" gate="G$1" pin="2"/>
@@
 </segment>
 </net>
-<net name="N$26" class="0">
+<net name="TX" class="0">
 <segment>
 <pinref part="JP13" gate="G$1" pin="1"/>
@@
 </segment>
 </net>
-<net name="N$29" class="0">
+<net name="RX" class="0">
 <segment>
 <pinref part="JP14" gate="G$1" pin="1"/>
@@
 </segment>
 </net>
-<net name="N$32" class="0">
+<net name="SDA" class="0">
 <segment>
 <pinref part="JP11" gate="G$1" pin="1"/>
@@
 </segment>
 </net>
-<net name="N$35" class="0">
+<net name="SCL" class="0">
 <segment>
 <pinref part="JP12" gate="G$1" pin="1"/>
@@
 </segment>
 </net>
-<net name="N$4" class="0">
+<net name="+3.3V" class="0">
 <segment>
 <pinref part="JP7" gate="G$1" pin="1"/>
@@
 </segment>
 </net>
-<net name="N$43" class="0">
+<net name="RST" class="0">
 <segment>
 <pinref part="JP2" gate="G$1" pin="1"/>
@@
 </segment>
 </net>
-<net name="N$48" class="0">
+<net name="SCK" class="0">
 <segment>
 <pinref part="JP4" gate="G$1" pin="1"/>
@@
 </segment>
 </net>
-<net name="N$2" class="0">
+<net name="+5V" class="0">
 <segment>
 <pinref part="MB1" gate="G$1" pin="+5V"/>

Commit message: Better Fritzing part thanks to Steve Lilley
Connections:
- net N$10 renamed R5
- net N$12 renamed L7
- net N$14 renamed R4
- net N$16 renamed L8
- net N$17 renamed L6
- net N$18 renamed R1
- net N$19 renamed R3
- net N$20 renamed R2
- net N$21 renamed R7
- net N$22 renamed L11
- net N$23 renamed R8
- net N$25 renamed L9
- net N$27 renamed R9
- net N$28 renamed R10
- net N$3 renamed L3
- net N$30 renamed R11
- net N$44 renamed L4
- net N$45 renamed L5
- net N$6 renamed L2
- net N$7 renamed L1
- net N$8 renamed R6
- net N$9 renamed L10
Changed lines of the file:
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@@
 </segment>
 </net>
-<net name="N$9" class="0">
+<net name="L10" class="0">
 <segment>
 <pinref part="U$4" gate="G$1" pin="P$1"/>
@@
 </segment>
 </net>
-<net name="N$12" class="0">
+<net name="L7" class="0">
 <segment>
 <pinref part="U$7" gate="G$1" pin="P$1"/>
@@
 </segment>
 </net>
-<net name="N$16" class="0">
+<net name="L8" class="0">
 <segment>
 <pinref part="U$8" gate="G$1" pin="P$1"/>
@@
 </segment>
 </net>
-<net name="N$17" class="0">
+<net name="L6" class="0">
 <segment>
 <pinref part="U$9" gate="G$1" pin="P$1"/>
@@
 </segment>
 </net>
-<net name="N$22" class="0">
+<net name="L11" class="0">
 <segment>
 <pinref part="U$5" gate="G$1" pin="P$1"/>
@@
 </segment>
 </net>
-<net name="N$25" class="0">
+<net name="L9" class="0">
 <segment>
 <pinref part="U$6" gate="G$1" pin="P$1"/>
@@
 </segment>
 </net>
-<net name="N$44" class="0">
+<net name="L4" class="0">
 <segment>
 <pinref part="U$1" gate="G$1" pin="P$1"/>
@@
 </segment>
 </net>
-<net name="N$45" class="0">
+<net name="L5" class="0">
 <segment>
 <pinref part="U$2" gate="G$1" pin="P$1"/>
@@
 </segment>
 </net>
-<net name="N$3" class="0">
+<net name="L3" class="0">
 <segment>
 <pinref part="U$3" gate="G$1" pin="P$1"/>
@@
 </segment>
 </net>
-<net name="N$6" class="0">
+<net name="L2" class="0">
 <segment>
 <pinref part="U$10" gate="G$1" pin="P$1"/>
@@
 </segment>
 </net>
-<net name="N$7" class="0">
+<net name="L1" class="0">
 <segment>
 <pinref part="U$11" gate="G$1" pin="P$1"/>
@@
 </segment>
 </net>
-<net name="N$8" class="0">
+<net name="R6" class="0">
 <segment>
 <pinref part="JP22" gate="G$1" pin="5"/>
@@
 </segment>
 </net>
-<net name="N$10" class="0">
+<net name="R5" class="0">
 <segment>
 <pinref part="JP23" gate="G$1" pin="5"/>
@@
 </segment>
 </net>
-<net name="N$14" class="0">
+<net name="R4" class="0">
 <segment>
 <pinref part="JP24" gate="G$1" pin="5"/>
@@
 </segment>
 </net>
-<net name="N$18" class="0">
+<net name="R1" class="0">
 <segment>
 <pinref part="JP27" gate="G$1" pin="5"/>
@@
 </segment>
 </net>
-<net name="N$19" class="0">
+<net name="R3" class="0">
 <segment>
 <pinref part="JP25" gate="G$1" pin="5"/>
@@
 </segment>
 </net>
-<net name="N$20" class="0">
+<net name="R2" class="0">
 <segment>
 <pinref part="JP26" gate="G$1" pin="5"/>
@@
 </segment>
 </net>
-<net name="N$21" class="0">
+<net name="R7" class="0">
 <segment>
 <pinref part="JP21" gate="G$1" pin="5"/>
@@
 </segment>
 </net>
-<net name="N$23" class="0">
+<net name="R8" class="0">
 <segment>
 <pinref part="JP20" gate="G$1" pin="5"/>
@@
 </segment>
 </net>
-<net name="N$27" class="0">
+<net name="R9" class="0">
 <segment>
 <pinref part="JP19" gate="G$1" pin="5"/>
@@
 </segment>
 </net>
-<net name="N$28" class="0">
+<net name="R10" class="0">
 <segment>
 <pinref part="JP18" gate="G$1" pin="5"/>
@@
 </segment>
 </net>
-<net name="N$30" class="0">
+<net name="R11" class="0">
 <segment>
 <pinref part="JP17" gate="G$1" pin="5"/>
